Commit message: update UR5 config

File: sdpf_bringup/config/ur5/end_effector.urdf.xacro (robot description, xacro)
@@ -4,5 +4,5 @@
   <link name="${prefix}ft_sensor"/>
   <joint name="${prefix}joint_tool0-ft_sensor" type="fixed">
-      <origin rpy="0 0 0" xyz="0 0 0.026"/>
+      <origin rpy="0 0 ${-3.1415/2}" xyz="0 0 0.026"/>
       <parent link="${prefix}${parent}"/>
       <child link="${prefix}ft_sensor"/>
@@ -11,5 +11,5 @@
   <link name="${prefix}interaction_point"/>
   <joint name="${prefix}ft_sensor-interaction_point" type="fixed">
-      <origin rpy="0 0 0" xyz="0 0 0.1"/>
+      <origin rpy="0 0 0" xyz="0 0 0.0"/>
       <parent link="${prefix}ft_sensor"/>
       <child link="${prefix}interaction_point"/>

File: sdpf_bringup/config/ur5/ft_sensor.ros2_control.xacro (robot description, xacro)
@@ -51,5 +51,5 @@
           <param name="alias">0</param>
           <param name="position">0</param>
-          <param name="slave_config">$(find sdpf_bringup)/config/ur5/ft_sensor_slave_config.yaml</param>
+          <param name="slave_config">$(find sdpf_bringup)/config/ur5/ft_sensor_ethercat_config.yaml</param>
         </ec_module>
         </xacro:unless>
